File: src/VisualEQ.kicad_sch (KiCad schematic)
At the start: 50 parts, among them J1 AudioJack3, J2 AudioJack3, J3 AudioJack3, J4 AudioPlug3, J5 AudioPlug3, J6 AudioPlug3, J8 Mini-DIN-6, J9 Mini-DIN-6, U1 ESP32-C3-WROOM-02, U2 MCP3208, U3 TL074, U4 TL074, U5 TLE2426xP

Commit message: Chanel fix
Connections:
- net CH4 is gone; now on net 5-: U2.5 (CH4)
- net +3V3: now also U1.1 (3V3)
- net 5-: no longer U2.6 (CH5)
- net 6-: now also U2.6 (CH5); no longer U2.7 (CH6), U4.8, U4.9
- net GND: now also U1.19 (GND), U1.9 (GND)
- new net CH6: U2.7 (CH6), U4.8, U4.9
Changed lines of the file:
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@@
 	(wire
 		(pts
+			(xy 218.44 143.51) (xy 217.17 143.51)
+		)
+		(stroke
+			(width 0)
+			(type default)
+		)
+	)
+	(wire
+		(pts
 			(xy 63.5 90.17) (xy 93.98 90.17)
 		)
@@
 	(wire
 		(pts
+			(xy 265.43 140.97) (xy 265.43 143.51)
+		)
+		(stroke
+			(width 0)
+			(type default)
+		)
+	)
+	(wire
+		(pts
 			(xy 62.23 52.07) (xy 63.5 52.07)
 		)
@@
 	(wire
 		(pts
+			(xy 265.43 143.51) (xy 264.16 143.51)
+		)
+		(stroke
+			(width 0)
+			(type default)
+		)
+	)
+	(wire
+		(pts
 			(xy 147.32 104.14) (xy 151.13 104.14)
 		)
@@
 	(wire
 		(pts
+			(xy 217.17 143.51) (xy 217.17 146.05)
+		)
+		(stroke
+			(width 0)
+			(type default)
+		)
+	)
+	(wire
+		(pts
 			(xy 167.64 143.51) (xy 186.69 143.51)
 		)
@@
 		)
 	)
-	(global_label "CH6"
+	(global_label "CH5"
 		(shape output)
 		(at 152.4 139.7 0)
@@
 		)
 	)
-	(global_label "CH5"
+	(global_label "CH4"
 		(shape output)
 		(at 152.4 127 0)
@@
 	)
 	(symbol
+		(lib_id "power:+3V3")
+		(at 265.43 140.97 0)
+		(unit 1)
+		(body_style 1)
+		(exclude_from_sim no)
+		(in_bom yes)
+		(on_board yes)
+		(in_pos_files yes)
+		(dnp no)
+		(fields_autoplaced yes)
+		(property "Reference" "#PWR017"
+			(at 265.43 144.78 0)
+			(hide yes)
+			(show_name no)
+			(do_not_autoplace no)
+			(effects
+				(font
+					(size 1.27 1.27)
+				)
+			)
+		)
+		(property "Value" "+3V3"
+			(at 265.43 135.89 0)
+			(show_name no)
+			(do_not_autoplace no)
+			(effects
+				(font
+					(size 1.27 1.27)
+				)
+			)
+		)
+		(property "Footprint" ""
+			(at 265.43 140.97 0)
+			(hide yes)
+			(show_name no)
+			(do_not_autoplace no)
+			(effects
+				(font
+					(size 1.27 1.27)
+				)
+			)
+		)
+		(property "Datasheet" ""
+			(at 265.43 140.97 0)
+			(hide yes)
+			(show_name no)
+			(do_not_autoplace no)
+			(effects
+				(font
+					(size 1.27 1.27)
+				)
+			)
+		)
+		(property "Description" "Power symbol creates a global label with name \"+3V3\""
+			(at 265.43 140.97 0)
+			(hide yes)
+			(show_name no)
+			(do_not_autoplace no)
+			(effects
+				(font
+					(size 1.27 1.27)
+				)
+			)
+		)
+		(pin "1"
+		)
+		(instances
+			(project "VisualEQ"
+				(path "/e1176a2b-c346-432a-9c8f-d15bd884be1d"
+					(reference "#PWR017")
+					(unit 1)
+				)
+			)
+		)
+	)
+	(symbol
 		(lib_id "Diode:1N4148")
 		(at 130.81 142.24 0)
@@
 		(in_pos_files yes)
 		(dnp no)
-		(fields_autoplaced yes)
 		(property "Reference" "U1"
-			(at 274.32 137.0898 90)
+			(at 221.742 160.02 90)
 			(show_name no)
 			(do_not_autoplace no)
@@
 		)
 		(property "Value" "ESP32-C3-WROOM-02"
-			(at 274.32 139.6298 90)
+			(at 231.902 157.734 90)
 			(show_name no)
 			(do_not_autoplace no)
@@
 					(unit 1)
 				)
+			)
+		)
+	)
+	(symbol
+		(lib_id "power:GND")
+		(at 217.17 146.05 0)
+		(unit 1)
+		(body_style 1)
+		(exclude_from_sim no)
+		(in_bom yes)
+		(on_board yes)
+		(in_pos_files yes)
+		(dnp no)
+		(fields_autoplaced yes)
+		(property "Reference" "#PWR016"
+			(at 217.17 152.4 0)
+			(hide yes)
+			(show_name no)
+			(do_not_autoplace no)
+			(effects
+				(font
+					(size 1.27 1.27)
+				)
+			)
+		)
+		(property "Value" "GND"
+			(at 217.17 151.13 0)
+			(show_name no)
+			(do_not_autoplace no)
+			(effects
+				(font
+					(size 1.27 1.27)
+				)
+			)
+		)
+		(property "Footprint" ""
+			(at 217.17 146.05 0)
+			(hide yes)
+			(show_name no)
+			(do_not_autoplace no)
+			(effects
+				(font
+					(size 1.27 1.27)
+				)
+			)
+		)
+		(property "Datasheet" ""
+			(at 217.17 146.05 0)
+			(hide yes)
+			(show_name no)
+			(do_not_autoplace no)
+			(effects
+				(font
+					(size 1.27 1.27)
+				)
+			)
+		)
+		(property "Description" "Power symbol creates a global label with name \"GND\" , ground"
+			(at 217.17 146.05 0)
+			(hide yes)
+			(show_name no)
+			(do_not_autoplace no)
+			(effects
+				(font
+					(size 1.27 1.27)
+				)
+			)
+		)
+		(pin "1"
+		)
+		(instances
+			(project "VisualEQ"
+				(path "/e1176a2b-c346-432a-9c8f-d15bd884be1d"
+					(reference "#PWR016")
+					(unit 1)
+				)
